File: STM32F405RG +  Gyro + I2C.sch (KiCad schematic (older format))
At the start: 62 parts, among them J1 USB_B_Micro, J2 USART_CONN, J3 SWD_CONN, J4 12V_CONN, Q1 AO3401A, SW1 SW_SPDT, U1 MP2359DJ-LF-Z, U2 MPU-6000, U3 USBLC6-2SC6, U4 STM32F405RGTx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

Commit message: Minor changes
Parts:
- J1: symbol Connector:USB_B_Micro -> STM32F405RG-+--Gyro-+-I2C-rescue:USB_B_Micro-Connector
- U1: symbol STM32F405RG-+--Gyro-+-I2C-rescue:MP2359DJ-LF-Z-OllieKiCadLibrary-STM32F405RG-+--Gyro-+-I2C-rescue-STM32F405RG-+--Gyro-+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 -> OllieKiCadLibrary:MP2359DJ-LF-Z
Changed lines of the file:
@@
 EESchema Schematic File Version 4
-EELAYER 30 0
+LIBS:STM32F405RG +  Gyro + I2C-cache
+EELAYER 29 0
 EELAYER END
 $Descr A3 16535 11693
@@
 $EndComp
 $Comp
-L STM32F405RG-+--Gyro-+-I2C-rescue:MP2359DJ-LF-Z-OllieKiCadLibrary-STM32F405RG-+--Gyro-+-I2C-rescue-STM32F405RG-+--Gyro-+-I2C-rescue U1
+L OllieKiCadLibrary:MP2359DJ-LF-Z U1
 U 1 1 6144594D
 P 5700 1750
@@
 VCAP1, VCAP2 and Decoupling capacitors needs to be ceramic
 $Comp
-L Connector:USB_B_Micro J1
+L STM32F405RG-+--Gyro-+-I2C-rescue:USB_B_Micro-Connector J1
 U 1 1 6148C1CA
 P 11900 5550
