File: STM32F405RG +  Gyro + I2C.sch (KiCad schematic (older format))
At the start: 62 parts, among them J1 USB_B_Micro, J2 USART_CONN, J3 SWD_CONN, J4 12V_CONN, Q1 AO3401A, SW1 SW_SPDT, U1 MP2359DJ-LF-Z, U2 MPU-6000, U3 USBLC6-2SC6, U4 STM32F405RGTx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

Commit message: Changes & PCB routing
Changed pin on LED, started routing signals and differential pairs
Parts:
- removed R12: 10k, Resistor_SMD:R_0402_1005Metric, symbol Device:R_Small
- J1: footprint USB Footprint Library:USB_Micro-B_GCT_USB3076-30-A -> USB Footprint Library:USB_Micro-B_Molex-105017-0001
- U3: symbol STM32F405RG-+--Gyro-+-I2C-rescue:USBLC6-2SC6-Power_Protection-STM32F405RG-+--Gyro-+-I2C-rescue-STM32F405RG-+--Gyro-+-I2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 -> Power_Protection:USBLC6-2SC6
Connections:
- net labels removed: BOOT1
- wire segments 188 -> 190
Changed lines of the file:
@@
 EESchema Schematic File Version 4
-LIBS:STM32F405RG +  Gyro + I2C-cache
-EELAYER 29 0
+EELAYER 30 0
 EELAYER END
 $Descr A3 16535 11693
@@
 Wire Wire Line
 	2450 1550 2450 1600
-$Comp
-L Connector_Generic:Conn_02x05_Odd_Even J3
-U 1 1 615724AF
-P 14150 7750
-F 0 "J3" H 14250 8350 50  0000 C CNN
-F 1 "SWD_CONN" H 14250 8250 50  0000 C CNN
-F 2 "Connector_PinSocket_1.27mm:PinSocket_2x05_P1.27mm_Vertical_SMD" H 14150 7750 50  0001 C CNN
-F 3 "~" H 14150 7750 50  0001 C CNN
-	1    14150 7750
-	1    0    0    -1
-$EndComp
 Wire Wire Line
 	7500 10250 7400 10250
@@
 	1    0    0    -1
 $EndComp
-NoConn ~ 13950 7850
-$Comp
-L power:+3V3 #PWR033
-U 1 1 615BFA1D
-P 13850 7550
-F 0 "#PWR033" H 13850 7400 50  0001 C CNN
-F 1 "+3V3" H 13750 7700 50  0000 L CNN
-F 2 "" H 13850 7550 50  0001 C CNN
-F 3 "" H 13850 7550 50  0001 C CNN
-	1    13850 7550
-	1    0    0    -1
-$EndComp
-Wire Wire Line
-	13850 7550 13950 7550
-Wire Wire Line
-	13950 7650 13900 7650
-Wire Wire Line
-	13900 7650 13900 7750
-Wire Wire Line
-	13900 7750 13950 7750
-$Comp
-L power:GND #PWR038
-U 1 1 615EA0AC
-P 13900 8000
-F 0 "#PWR038" H 13900 7750 50  0001 C CNN
-F 1 "GND" H 13905 7827 50  0000 C CNN
-F 2 "" H 13900 8000 50  0001 C CNN
-F 3 "" H 13900 8000 50  0001 C CNN
-	1    13900 8000
-	1    0    0    -1
-$EndComp
-Wire Wire Line
-	13900 7750 13900 7950
-Connection ~ 13900 7750
-Wire Wire Line
-	13900 7950 13950 7950
-Connection ~ 13900 7950
-Wire Wire Line
-	13900 7950 13900 8000
 Text GLabel 5300 8250 2    50   Input ~ 0
 SWDIO
@@
 USB_CONN_D+
 $Comp
-L STM32F405RG-+--Gyro-+-I2C-rescue:USBLC6-2SC6-Power_Protection-STM32F405RG-+--Gyro-+-I2C-rescue-STM32F405RG-+--Gyro-+-I2C-rescue U3
+L Power_Protection:USBLC6-2SC6 U3
 U 1 1 613CB340
 P 14550 5550
@@
 Wire Wire Line
 	7350 2800 7350 2850
-Text GLabel 5300 8850 2    50   Input ~ 0
-BOOT1
-Wire Wire Line
-	5300 8850 5200 8850
-Text GLabel 7350 7900 0    50   Input ~ 0
-BOOT1
-$Comp
-L power:GND #PWR039
-U 1 1 614B62CE
-P 7450 8250
-F 0 "#PWR039" H 7450 8000 50  0001 C CNN
-F 1 "GND" H 7455 8077 50  0000 C CNN
-F 2 "" H 7450 8250 50  0001 C CNN
-F 3 "" H 7450 8250 50  0001 C CNN
-	1    7450 8250
-	1    0    0    -1
-$EndComp
 Wire Notes Line
 	6750 6900 6750 8500
-$Comp
-L Device:R_Small R12
-U 1 1 614DE8D8
-P 7450 8100
-F 0 "R12" H 7300 8150 50  0000 C CNN
-F 1 "10k" H 7300 8050 50  0000 C CNN
-F 2 "Resistor_SMD:R_0402_1005Metric" H 7450 8100 50  0001 C CNN
-F 3 "~" H 7450 8100 50  0001 C CNN
-	1    7450 8100
-	1    0    0    -1
-$EndComp
-Wire Wire Line
-	7450 7900 7450 8000
-Wire Wire Line
-	7450 8200 7450 8250
-Wire Wire Line
-	7350 7900 7450 7900
 Text Notes 6650 3550 0    39   Italic 0
 FB (Feedback voltage) needs to be between 0.790 V and 0.830 V\n\n(15k+270)/(47k+15k+270) * 3.3V = 0.80923 V
@@
 F 0 "J1" H 11957 6017 50  0000 C CNN
 F 1 "USB_B_Micro" H 11957 5926 50  0000 C CNN
-F 2 "USB Footprint Library:USB_Micro-B_GCT_USB3076-30-A" H 12050 5500 50  0001 C CNN
+F 2 "USB Footprint Library:USB_Micro-B_Molex-105017-0001" H 12050 5500 50  0001 C CNN
 F 3 "~" H 12050 5500 50  0001 C CNN
 	1    11900 5550
@@
 	1    0    0    -1
 $EndComp
-Text GLabel 3700 9850 0    50   Input ~ 0
+Text GLabel 5300 9150 2    50   Input ~ 0
 LED
 Wire Wire Line
-	3700 9850 3800 9850
+	5300 9150 5200 9150
 Connection ~ 2450 2000
 Wire Wire Line
@@
 	0    1    -1   0
 $EndComp
+Wire Wire Line
+	14550 5050 14550 5150
+Wire Wire Line
+	14950 5450 15050 5450
+Wire Wire Line
+	14950 5650 15050 5650
+Wire Wire Line
+	14550 5950 14550 6050
+Wire Wire Line
+	14050 5650 14150 5650
+Wire Wire Line
+	14050 5450 14150 5450
+Wire Wire Line
+	13900 7950 13900 8000
+Connection ~ 13900 7950
+Wire Wire Line
+	13900 7950 13950 7950
+Connection ~ 13900 7750
+Wire Wire Line
+	13900 7750 13900 7950
+$Comp
+L power:GND #PWR038
+U 1 1 615EA0AC
+P 13900 8000
+F 0 "#PWR038" H 13900 7750 50  0001 C CNN
+F 1 "GND" H 13905 7827 50  0000 C CNN
+F 2 "" H 13900 8000 50  0001 C CNN
+F 3 "" H 13900 8000 50  0001 C CNN
+	1    13900 8000
+	1    0    0    -1
+$EndComp
+Wire Wire Line
+	13900 7750 13950 7750
+Wire Wire Line
+	13900 7650 13900 7750
+Wire Wire Line
+	13950 7650 13900 7650
+Wire Wire Line
+	13850 7550 13950 7550
+$Comp
+L power:+3V3 #PWR033
+U 1 1 615BFA1D
+P 13850 7550
+F 0 "#PWR033" H 13850 7400 50  0001 C CNN
+F 1 "+3V3" H 13750 7700 50  0000 L CNN
+F 2 "" H 13850 7550 50  0001 C CNN
+F 3 "" H 13850 7550 50  0001 C CNN
+	1    13850 7550
+	1    0    0    -1
+$EndComp
+NoConn ~ 13950 7850
+$Comp
+L Connector_Generic:Conn_02x05_Odd_Even J3
+U 1 1 615724AF
+P 14150 7750
+F 0 "J3" H 14250 8350 50  0000 C CNN
+F 1 "SWD_CONN" H 14250 8250 50  0000 C CNN
+F 2 "Connector_PinSocket_1.27mm:PinSocket_2x05_P1.27mm_Vertical_SMD" H 14150 7750 50  0001 C CNN
+F 3 "~" H 14150 7750 50  0001 C CNN
+	1    14150 7750
+	1    0    0    -1
+$EndComp
 $EndSCHEMATC

Commit message: Fixed layout and added text to silkscreen
Parts:
- J1: symbol STM32F405RG-+--Gyro-+-I2C-rescue:USB_B_Micro-Connector -> Connector:USB_B_Micro
- U3: symbol Power_Protection:USBLC6-2SC6 -> STM32F405RG-+--Gyro-+-I2C-rescue:USBLC6-2SC6-Power_Protection
Connections:
- no-connect marks 6 -> 41
Changed lines of the file:
@@
 EESchema Schematic File Version 4
-EELAYER 30 0
+LIBS:STM32F405RG +  Gyro + I2C-cache
+EELAYER 29 0
 EELAYER END
 $Descr A3 16535 11693
@@
 U 1 1 6138CF9E
 P 4500 8550
-F 0 "U4" H 5100 6750 50  0000 C CNN
-F 1 "STM32F405RGTx" H 5150 6650 50  0000 C CNN
+F 0 "U4" H 4500 6661 50  0000 C CNN
+F 1 "STM32F405RGTx" H 4500 6570 50  0000 C CNN
 F 2 "Package_QFP:LQFP-64_10x10mm_P0.5mm" H 3900 6850 50  0001 R CNN
 F 3 "http://www.st.com/st-web-ui/static/active/en/resource/technical/document/datasheet/DM00037051.pdf" H 4500 8550 50  0001 C CNN
@@
 Text Notes 6700 10800 0    50   ~ 0
 Pull-up resistors are needed for I2C to \nensure the logical state. \nShould be in range 2k to 10k
-Text GLabel 3700 9050 0    50   Input ~ 0
+Text GLabel 3700 9950 0    50   Input ~ 0
 GYRO_INT
 Wire Wire Line
-	3700 9050 3800 9050
+	3700 9950 3800 9950
 Text GLabel 14150 2250 2    50   Input ~ 0
 GYRO_INT
@@
 USB_CONN_D+
 $Comp
-L Power_Protection:USBLC6-2SC6 U3
+L STM32F405RG-+--Gyro-+-I2C-rescue:USBLC6-2SC6-Power_Protection U3
 U 1 1 613CB340
 P 14550 5550
@@
 VCAP1, VCAP2 and Decoupling capacitors needs to be ceramic
 $Comp
-L STM32F405RG-+--Gyro-+-I2C-rescue:USB_B_Micro-Connector J1
+L Connector:USB_B_Micro J1
 U 1 1 6148C1CA
 P 11900 5550
@@
 	1    0    0    -1
 $EndComp
+NoConn ~ 5200 8650
+NoConn ~ 5200 8750
+NoConn ~ 5200 8850
+NoConn ~ 5200 9050
+NoConn ~ 5200 8450
+NoConn ~ 5200 9250
+NoConn ~ 5200 9550
+NoConn ~ 5200 9850
+NoConn ~ 5200 9950
+NoConn ~ 5200 10050
+NoConn ~ 5200 10150
+NoConn ~ 3800 10150
+NoConn ~ 3800 10050
+NoConn ~ 3800 9850
+NoConn ~ 3800 9750
+NoConn ~ 3800 9650
+NoConn ~ 3800 9550
+NoConn ~ 3800 9450
+NoConn ~ 3800 9350
+NoConn ~ 3800 9250
+NoConn ~ 3800 9150
+NoConn ~ 3800 9050
+NoConn ~ 3800 8950
+NoConn ~ 3800 8850
+NoConn ~ 3800 8750
+NoConn ~ 3800 8650
+NoConn ~ 3800 8450
+NoConn ~ 5200 7950
+NoConn ~ 5200 7850
+NoConn ~ 5200 7750
+NoConn ~ 5200 7650
+NoConn ~ 5200 7550
+NoConn ~ 5200 7450
+NoConn ~ 5200 7350
+NoConn ~ -100 10000
 $EndSCHEMATC

Commit message: Changes
FIX: Changed SWD connector from socket to header
Parts:
- J1: symbol Connector:USB_B_Micro -> STM32F405RG-+--Gyro-+-I2C-rescue:USB_B_Micro-Connector
- J3: footprint Connector_PinSocket_1.27mm:PinSocket_2x05_P1.27mm_Vertical_SMD -> Connector_PinHeader_1.27mm:PinHeader_2x05_P1.27mm_Vertical_SMD
Changed lines of the file:
@@
 EESchema Schematic File Version 4
-LIBS:STM32F405RG +  Gyro + I2C-cache
-EELAYER 29 0
+EELAYER 30 0
 EELAYER END
 $Descr A3 16535 11693
@@
 VCAP1, VCAP2 and Decoupling capacitors needs to be ceramic
 $Comp
-L Connector:USB_B_Micro J1
+L STM32F405RG-+--Gyro-+-I2C-rescue:USB_B_Micro-Connector J1
 U 1 1 6148C1CA
 P 11900 5550
@@
 F 0 "J3" H 14250 8350 50  0000 C CNN
 F 1 "SWD_CONN" H 14250 8250 50  0000 C CNN
-F 2 "Connector_PinSocket_1.27mm:PinSocket_2x05_P1.27mm_Vertical_SMD" H 14150 7750 50  0001 C CNN
+F 2 "Connector_PinHeader_1.27mm:PinHeader_2x05_P1.27mm_Vertical_SMD" H 14150 7750 50  0001 C CNN
 F 3 "~" H 14150 7750 50  0001 C CNN
 	1    14150 7750

Commit message: Added BOM file
Parts:
- J1: symbol STM32F405RG-+--Gyro-+-I2C-rescue:USB_B_Micro-Connector -> STM32F405RG-+--Gyro-+-I2C-rescue:USB_B_Micro-Connector-STM32F405RG-+--Gyro-+-I2C-rescue
- U3: symbol STM32F405RG-+--Gyro-+-I2C-rescue:USBLC6-2SC6-Power_Protection -> Power_Protection:USBLC6-2SC6
Changed lines of the file:
@@
 Text GLabel 15050 5650 2    50   Input ~ 0
 USB_CONN_D+
-$Comp
-L STM32F405RG-+--Gyro-+-I2C-rescue:USBLC6-2SC6-Power_Protection U3
-U 1 1 613CB340
-P 14550 5550
-F 0 "U3" H 14950 6100 50  0000 C CNN
-F 1 "USBLC6-2SC6" H 14950 6000 50  0000 C CNN
-F 2 "Package_TO_SOT_SMD:SOT-23-6" H 13800 5950 50  0001 C CNN
-F 3 "http://www2.st.com/resource/en/datasheet/CD00050750.pdf" H 14750 5900 50  0001 C CNN
-	1    14550 5550
-	1    0    0    -1
-$EndComp
 Wire Notes Line
 	15900 4700 15900 6400
@@
 VCAP1, VCAP2 and Decoupling capacitors needs to be ceramic
 $Comp
-L STM32F405RG-+--Gyro-+-I2C-rescue:USB_B_Micro-Connector J1
+L STM32F405RG-+--Gyro-+-I2C-rescue:USB_B_Micro-Connector-STM32F405RG-+--Gyro-+-I2C-rescue J1
 U 1 1 6148C1CA
 P 11900 5550
@@
 NoConn ~ 5200 7350
 NoConn ~ -100 10000
+$Comp
+L Power_Protection:USBLC6-2SC6 U3
+U 1 1 613CB340
+P 14550 5550
+F 0 "U3" H 14950 6100 50  0000 C CNN
+F 1 "USBLC6-2SC6" H 14950 6000 50  0000 C CNN
+F 2 "Package_TO_SOT_SMD:SOT-23-6" H 13800 5950 50  0001 C CNN
+F 3 "http://www2.st.com/resource/en/datasheet/CD00050750.pdf" H 14750 5900 50  0001 C CNN
+	1    14550 5550
+	1    0    0    -1
+$EndComp
 $EndSCHEMATC

Commit message: Changed gyroscope, added gerber and assembly files
-Changed Gyroscope from MPU-6000 to MPU-6050
-Added Gerber and Assembly files
Parts:
- added C20: 10uF, Capacitor_SMD:C_1206_3216Metric, symbol Device:C_Small
- added C21: 10nF, Capacitor_SMD:C_0603_1608Metric, symbol Device:C_Small
- C1: LCSC (none) -> C13585
- C10, C9: LCSC (none) -> C23630
- C11: LCSC (none) -> C19666
- C12, C13, C14, C15, C16, C19, C6: LCSC (none) -> C1525
- C17: LCSC (none) -> C52923
- C18: LCSC (none) -> C15195
- C2: LCSC (none) -> C57112
- C3: value 22uF -> 10uF; LCSC (none) -> C13585
- C4, C5: LCSC (none) -> C32949
- C7: LCSC (none) -> C14663
- C8: LCSC (none) -> C1604
- D1, D2: LCSC (none) -> C8598
- D3: LCSC (none) -> C2286
- D4, D5, D6, D7: LCSC (none) -> C72041
- D8: LCSC (none) -> C72038
- F1, R5: LCSC (none) -> C369159
- FB1: LCSC (none) -> C1017
- L1: LCSC (none) -> C408347
- L2: LCSC (none) -> C26443
- Q1: LCSC (none) -> C15127
- R1: LCSC (none) -> C25808
- R10, R11, R8, R9: LCSC (none) -> C25092
- R13: value 68 -> 47; LCSC (none) -> C25118
- R14, R15: LCSC (none) -> C25879
- R16, R17, R18, R19: LCSC (none) -> C25867
- R2: LCSC (none) -> C25819
- R20: LCSC (none) -> C21190
- R3: LCSC (none) -> C23254
- R4: LCSC (none) -> C22809
- R6: LCSC (none) -> C22966
- R7: LCSC (none) -> C25744
- U1: LCSC (none) -> C14259
- U2: value MPU-6000 -> MPU-6050; symbol Sensor_Motion:MPU-6000 -> Sensor_Motion:MPU-6050; LCSC (none) -> C24112
- U3: LCSC (none) -> C7519
- U4: LCSC (none) -> C15742
- Y1: LCSC (none) -> C13738
Connections:
- net +3V3: now also C20.1, C21.1
- net GND: now also C20.2, C21.2
Other:
- note added: "Gyroscope MPU6050\n"
- note added: "INT (interrupt) pin which is an interrupt digital output pin and used to \ngive indication to the MCU that data is available to read from the MPU6050.\n\nFSYNC is used to sync the MPU6050 with a videocamera etc. \nIf unused, connect to ground according to datasheet. \n\nCLKIN is optional external reference clock input. If unused, connect to ground according to datasheet."
- note removed: "Gyroscope MPU6000"
- note removed: "INT (interrupt) pin which is an interrupt digital output pin and used to \ngive indication to the MCU that data is available to read from the MPU6000.\n\nFSYNC is used to sync the MP6000 with a videocamera etc. \nIf unused, connect to ground according to datasheet. \n\nCLKIN is optional external reference clock input. If unused, connect to ground according to datasheet."
- moved on the sheet: C6
